File: KiCAD/a8-proto-card/cad-files/Connectors.kicad_sch (KiCad schematic)
At the start: 11 parts, among them J1 ORESAT-DEBUG-CONNECTOR-CARD, J4 TFM-120-01-L-D-RA, J6 J-MOLEX-SMPM-73300-003X

Commit message: removed page 6; edited connectors, PWR and SD reader schematic
Other:
- moved on the sheet: J1, J4, J6, TP183, TP184, TP58, TP59, TP60, TP61, TP62
