File: KiCAD/a8-proto-card/cad-files/OSD3358_PWR,_ETC._%3a_SIP_A,_E,_F.kicad_sch (KiCad schematic)
At the start: 53 parts, among them Q1 MMBT2907, U10 TLVH431, U18 RCLAMP0504FB, U4 SN74LVC1G07DCK, U7 OSD3358-512M-BSM

Commit message: removed page 6; edited connectors, PWR and SD reader schematic
Connections:
- net GND: now also U7.D8 (DGND@1), U7.D9 (DGND@2), U7.E10 (DGND@8), U7.E11 (DGND@9), U7.E12 (DGND@10), U7.E5 (DGND@3), U7.E6 (DGND@4), U7.E7 (DGND@5), U7.E8 (DGND@6), U7.E9 (DGND@7), U7.F12 (DGND@12), U7.F5 (DGND@11), U7.G12 (DGND@14), U7.G5 (DGND@13), U7.H12 (DGND@17), U7.H13 (DGND@18), U7.H4 (DGND@15), U7.H5 (DGND@16), U7.J12 (DGND@21), U7.J13 (DGND@22), U7.J4 (DGND@19), U7.J5 (DGND@20), U7.K12 (DGND@24), U7.K5 (DGND@23), U7.L12 (DGND@26), U7.L5 (DGND@25), U7.M10 (DGND@32), U7.M11 (DGND@33), U7.M12 (DGND@34), U7.M5 (DGND@27), U7.M6 (DGND@28), U7.M7 (DGND@29), U7.M8 (DGND@30), U7.M9 (DGND@31), U7.N8 (DGND@35), U7.N9 (DGND@36); no longer U7.F8 (SYS_VDD3_3P3V@1), U7.G8 (SYS_VDD3_3P3V@2), U7.G9 (VDDSHV5), U7.H8 (SYS_VDD3_3P3V@4), U7.H9 (VDDSHV6), U7.J7 (SYS_VDD3_3P3V@5), U7.J9 (VDDSHV1), U7.K8 (SYS_VDD3_3P3V@7), U7.K9 (VDDSHV2), U7.L4 (PMIC_NWAKEUP), U7.L8 (SYS_VDD3_3P3V@8), U7.L9 (VDDSHV3), U7.M13 (PMIC_NRESET), U7.N11 (PMIC_PWR_EN), U7.N4 (PMIC_LDO_PGOOD), U7.N5 (RTC_PWRONRSTN), U7.T11 (PMIC_PB_IN)
- net at TP172.1: now also U7.D12 (NC@1)
- net at TP150.1: now also U7.J6 (NC@2)
- net at TP154.1: now also U7.G4 (VDD_CORE)
- net at TP156.1: now also U7.F4 (VDDS_DDR)
- net at TP166.1: now also U7.G13 (VDDS_PLL)
- net at TP160.1: now also U7.F13 (VDD_MPU)
- net at TP157.1: now also U7.H6 (VPP)
- net at TP173.1: now also U7.D5 (CAP_VDD_RTC)
- net at TP145.1: now also U7.K4 (NC@3)
Other:
- company: (none) -> PSAS
- title: (none) -> OreSat DxWiFi: OSD Power/Misc
- moved on the sheet: C13, C14, C18, C41, D1, JP101, JP104, Q1, R1, R15, R23, R28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
