File: KiCAD/a8-proto-card/cad-files/OSD3358_SD,_eMMC%3a_SIP_C,_D.kicad_sch (KiCad schematic)
At the start: 84 parts, among them J7 DM3BT-DSF-PEJS, U11 TCAN330, U17 25AAXX, U3 THGBMJG7C2LBAU8, U7 OSD3358-512M-BSM

Commit message: removed page 6; edited connectors, PWR and SD reader schematic
Connections:
- net PA_ENABLE: now also U7.H16 (MII1_TX_CLK)
- net UART0_RX: now also U7.A12 (UART0_RXD)
- net UART0_TX: now also U7.B12 (UART0_TXD)
- net at TP180.1: now also U7.C5 (ECAP0_IN_PWM0_OUT)
- net at TP127.1: now also U7.N2 (GPMC_WEN)
- net at TP123.1: now also U7.P5 (GPMC_AD9)
- net at JP108.2: now also U7.H3 (LCD_DATA3)
- net at TP101.1: now also U7.T13 (GPMC_A3)
- net at TP122.1: now also U7.P3 (GPMC_CSN0)
- net at JP109.2: now also U7.H2 (LCD_DATA4)
- net at R9.1 (11), U3.B3 (D4): now also U7.T2 (GPMC_AD4)
- net at R9.2 (22), U3.B2 (D3): now also U7.T3 (GPMC_AD3)
- net at R9.3 (33), U3.A5 (D2): now also U7.R1 (GPMC_AD2)
- net at R9.4 (44), U3.B6 (D7): now also U7.R4 (GPMC_AD7)
- net at R9.6 (66), U3.M5 (CMD): now also U7.P1 (GPMC_CSN2)
- net at R9.7 (77), U3.A3 (D0): now also U7.R3 (GPMC_AD0)
- net at R9.8 (88), U3.A4 (D1): now also U7.R2 (GPMC_AD1)
- net at R9.9 (99), U3.B4 (D5): now also U7.T1 (GPMC_AD5)
- net at TP105.1: now also U7.T5 (GPMC_AD11)
- net at TP120.1: now also U7.R6 (GPMC_AD13)
- net at TP126.1: now also U7.P12 (GPMC_A2)
- net at TP143.1: now also U7.J14 (RMII1_REF_CLK)
- net at TP114.1: now also U7.P15 (GPMC_WAIT0)
- net at R10.1 (11), U3.B5 (D6): now also U7.P4 (GPMC_AD6)
- net at R10.2 (22), U3.K5 (~{RST}): now also U7.R13 (GPMC_A4)
- net at R10.9 (99), U3.M6 (SCK): now also U7.P2 (GPMC_CSN1)
- net at TP159.1: now also U7.E1 (LCD_AC_BIAS_EN)
- net at R25.4 (44): now also U7.H1 (LCD_DATA5)
- net at R25.7 (77): now also U7.J3 (LCD_DATA6)
- net at TP115.1: now also U7.R5 (GPMC_AD10)
- net at U17.1 (~{CS}): now also U7.A14 (SPI0_CS0)
- net at U17.2 (MISO): now also U7.B13 (SPI0_D0)
- net at U17.5 (MOSI): now also U7.B14 (SPI0_D1)
- net at U17.6 (SCK): now also U7.A13 (SPI0_SCLK)
- net at TP158.1: now also U7.E13 (MDIO)
- net at TP131.1: now also U7.N3 (GPMC_BEN0_CLE)
- net at TP125.1: now also U7.N14 (GPMC_BEN1)
- net at R24.2 (22): now also U7.L1 (LCD_DATA14)
- net at R3.1: now also U7.T14 (GPMC_A6)
- net at TP137.1: now also U7.H15 (MII1_TXD0)
- net at R26.1 (11): now also U7.M3 (LCD_DATA15)
- net at R26.2 (22): now also U7.L3 (LCD_DATA12)
- net at R26.3 (33): now also U7.K2 (LCD_DATA10)
- net at R26.4 (44): now also U7.J1 (LCD_DATA8)
- net at R26.6 (66): now also U7.J2 (LCD_DATA7)
- net at R26.7 (77): now also U7.K3 (LCD_DATA9)
- net at R26.8 (88): now also U7.K1 (LCD_DATA11)
- net at R26.9 (99): now also U7.L2 (LCD_DATA13)
- net at R4.1: now also U7.R14 (GPMC_A7)
- net at U11.1 (TXD): now also U7.A11 (UART1_RXD)
- net at U11.4 (RXD): now also U7.B11 (UART1_TXD)
- net at TP135.1: now also U7.G16 (MII1_TXD2)
- net at TP134.1: now also U7.M1 (GPMC_ADVN_ALE)
- net at JP106.2: now also U7.G2 (LCD_DATA1)
- net at TP108.1: now also U7.T15 (GPMC_A9)
- net at J7.CD (CD#), R8.6 (66), TP22.1: now also U7.C14 (SPI0_CS1)
- net at JP105.2: now also U7.G3 (LCD_DATA0)
- net at TP174.1: now also U7.D13 (MDC)
- net at TP100.1: now also U7.T12 (GPMC_A0)
- net at TP149.1: now also U7.H14 (MII1_TXD1)
- net at J7.1 (DAT2), R8.2 (22): now also U7.C16 (MMC0_DAT2)
- net at J7.3 (CMD/DI), R8.3 (33): now also U7.B16 (MMC0_CMD)
- net at J7.7 (DAT0/DO), R8.4 (44): now also U7.A16 (MMC0_DAT0)
- net at J7.8 (DAT1), R8.7 (77): now also U7.A15 (MMC0_DAT1)
- net at J7.5 (CLK), R8.8 (88): now also U7.B15 (MMC0_CLK)
- net at J7.2 (DAT3/CS), R8.9 (99): now also U7.C15 (MMC0_DAT3)
- net at R2.1: now also U7.P13 (GPMC_A5)
- net at TP124.1: now also U7.P6 (GPMC_AD12)
- net at TP30.1: now also U7.A4 (XDMA_EVENT_INTR0)
- net at TP153.1: now also U7.F3 (LCD_VSYNC)
- net at TP103.1: now also U7.T16 (GPMC_A11)
- net at TP118.1: now also U7.R12 (GPMC_A1)
- net at JP107.2, U$1.P$2 (2): now also U7.G1 (LCD_DATA2)
- net at TP111.1: now also U7.R16 (GPMC_WPN)
- net at TP148.1: now also U7.G14 (MII1_TX_EN)
- net at TP104.1: now also U7.T4 (GPMC_AD8)
- net at R5.1: now also U7.P14 (GPMC_A8)
- net at TP117.1: now also U7.R15 (GPMC_A10)
- net at TP152.1: now also U7.F2 (LCD_HSYNC)
- net at TP178.1: now also U7.C13 (UART0_RTSN)
- net at TP106.1: now also U7.T7 (GPMC_CLK)
- net at TP162.1: now also U7.F1 (LCD_PCLK)
- net at TP107.1: now also U7.R7 (GPMC_CSN3)
- net at TP128.1: now also U7.N1 (GPMC_OEN_REN)
- net at TP177.1: now also U7.C12 (UART0_CTSN)
Other:
- moved on the sheet: C10, C11, C12, C2, C3, C31, C40, C5, C6, C8, C9, J7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
