File: KiCAD/a8-proto-card/cad-files/OSD3358_USB,_JTAG,_XTAL,_etc_%3a_SIP_B.kicad_sch (KiCad schematic)
At the start: 91 parts, among them J10 SM06B-SRSS-TB(LF)(SN), J8 FTSH-105-XX-X-DV-K, U1 RCLAMP0504FB, U2 TUSB2046IBVF, U20 TPS2041BQDBVRQ1, U21 TPS2041BQDBVRQ1, U7 OSD3358-512M-BSM, U9 TPS2041BQDBVRQ1, Y1 24MHz, Y2 ABS07-32.768KHZ-T, Y3 6MHz

Commit message: removed page 6; edited connectors, PWR and SD reader schematic
Connections:
- net 1.8V-A: now also U7.A7 (SYS_ADC_1P8V), U7.B7 (VREFP), U7.N13 (PMIC_MUX_IN)
- net GND: now also U7.A9 (AGND_ADC), U7.B9 (VREFN)
- net OSC0_GND: now also U7.N15 (OSC0_GND)
- net OSC0_IN: now also U7.P16 (OSC0_IN)
- net OSC0_OUT: now also U7.N16 (OSC0_OUT)
- net PA_THERMISTOR: now also U7.C9 (AIN6)
- net USB_DEV_N: now also U7.K16 (USB0_DM)
- net USB_DEV_P: now also U7.K15 (USB0_DP)
- net VIN_USB: now also U7.J16 (USB0_VBUS)
- net at R22.1: now also U7.E2 (EMU0)
- net at TP12.1: now also U7.M14 (USB1_DRVVBUS)
- net at R19.2, TP31.1: now also U7.D3 (TRSTN)
- net at TP181.1: now also U7.B6 (AIN2)
- net at TP139.1: now also U7.J15 (USB0_DRVVBUS)
- net at TP176.1: now also U7.C7 (AIN4)
- net at TP175.1: now also U7.C6 (AIN3)
- net at U2.1 (DP0): now also U7.L15 (USB1_DP)
- net at U2.2 (DM0): now also U7.L16 (USB1_DM)
- net at C29.1, R27.1, Y2.P$1: now also U7.A5 (OSC1_OUT)
- net at C30.1, R27.2, Y2.P$2: now also U7.A6 (OSC1_IN)
- net at J8.2 (SWDIO/TMS): now also U7.D2 (TMS)
- net at J8.4 (SWDCLK/TCK): now also U7.D1 (TCK)
- net at J8.6 (SWO/TDO): now also U7.C2 (TDO)
- net at J8.8 (NC/TDI): now also U7.C1 (TDI)
- net at TP141.1: now also U7.K13 (USB0_CE)
- net at TP169.1: now also U7.C8 (AIN5)
- net at JP100.1: now also U7.L14 (USB1_ID)
- net at TP144.1: now also U7.L13 (USB1_CE)
- net at TP39.1: now also U7.A8 (AIN0)
- net at R20.1: now also U7.E3 (EMU1)
- net at C29.2, C30.2: now also U7.B5 (OSC1_GND)
- net at TP38.1: now also U7.B8 (AIN1)
- net at TP138.1: now also U7.K14 (USB0_ID)
- new net: U7.D6 (PMIC_MUX_OUT), U7.D7 (AIN7)
Other:
- moved on the sheet: C1, C19, C22, C24, C25, C26, C27, C28, C29, C30, C4, C42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
