File: KiCAD/a8-proto-card/cad-files/Power.kicad_sch (KiCad schematic)
At the start: 98 parts, among them Q2 PMV45EN2R, Q3 DMP2240UDM, Q4 PMV45EN2R, Q5 DMP3050LVT-7, Q6 DMP3050LVT-7, U12 MIC842LYC5, U13 MIC842LYC5, U14 MAX4211FETE, U15 TPS62112, U16 MAX7310ATE, U5 TPS62112

Commit message: removed page 6; edited connectors, PWR and SD reader schematic
Connections:
- net PEN-SDA-FILT: now also Q3.4 (D); no longer Q3.6 (D)
- net at R43.2: now also Q3.3 (G); no longer Q3.1 (G)
- net at R41.2: now also Q3.2 (S); no longer Q3.5 (S)
Other:
- note added: "POWER"
- note added: "should it be removed"
- company: (none) -> PSAS
- title: (none) -> OreSat DxWiFi: OPD v4.1
- moved on the sheet: C16, C17, C20, C32, C33, C34, C35, C36, C37, C38, C39, C44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
