File: KiCAD/f0-proto-card/Connectors.kicad_sch (KiCad schematic)
At the start: 13 parts, among them J1 J-SAMTEC-TFM-110-X1-XXX-D-RA, J2 U.FL, J3 U.FL, J4 U.FL, J6 J-SAMTEC-TFM-120-X1-XXX-D-RA

Commit message: Some design review changes for protocard v5.0
Other:
- note removed: "4.2"
- note removed: "OreSat Proto-Card"
- title: (none) -> oresat-proto-card
- moved on the sheet: CM1, CM2, CM3, J1, J2, J3, J4, J6, JP2, JP9
