File: KiCAD/f0-proto-card/oresat-proto-card.kicad_sch (KiCad schematic)
At the start: 0 parts

Commit message: Some design review changes for protocard v5.0
Other:
- title: (none) -> oresat-proto-card
Changed lines of the file:
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@@
 (kicad_sch (version 20230121) (generator eeschema)
   (paper "User" 469.9 317.627)
+  (title_block
+    (title "oresat-proto-card")
+    (date "2024-02-25")
+    (rev "5.0")
+  )
   (sheet (at 25.4 25.4) (size 12.7 3.81) (fields_autoplaced)
     (stroke (width 0) (type solid))
