File: KiCAD/f0-proto-card/Power.kicad_sch (KiCad schematic)
At the start: 84 parts, among them Q1 MOSFET-PCH-SOT23-6, Q2 MOSFET-PCH-SOT23-6, Q7 MOSFET-PCH-SOT23-6, Q8 PMV45EN, Q9 PMV45EN, U10 TPS6211X, U11 MIC842LYC5, U12 MIC842LYC5, U2 MAX7310, U3 TS5A21366DCUR, U6 MAX4211

Commit message: Some design review changes for protocard v5.0
Parts:
- added C4: 470n, oresat-passives:0603-C-NOSILK, symbol oresat-acs-card-eagle-import:C-EU0603-C-NOSILK
- added C5: 10n, oresat-passives:0603-C-NOSILK, symbol oresat-acs-card-eagle-import:C-EU0603-C-NOSILK
- added R4, R5: RC0603FR-0710KL, oresat-passives:0603-C-NOSILK, symbol oresat-acs-card-eagle-import:R-US_0603-C-NOSILK
- added R6, R7: 0, oresat-proto-card:.0603-C-NOSILK, symbol oresat-proto-card-eagle-import:R-US_0603-C-NOSILK
- R39, R40, R45, R46, R52, R53, R54, R55, R56, R57, R58, R59, R67, R69: now not fitted
- U10: value TPS6211X -> TPS62111RSA
Connections:
- net CB_CTRL: now also R5.1; no longer Q2.3 (G), R70.1
- net PB6/SCL: now also R7.1; no longer U2.4 (IO0)
- net PB7/SDA: now also R6.1; no longer U2.5 (IO1)
- net VBUSP: now also C4.2
- net at Q2.4 (S), R64.2, R70.2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: now also C5.2
- new net: C5.1, Q2.3 (G), R4.2, R5.2, R70.1
- new net: R6.2, U2.5 (IO1)
- new net: C4.1, R4.1
- new net: R7.2, U2.4 (IO0)
Other:
- note added: "Circuit breaker switch with ~10 ms soft start"
- note removed: "4.2"
- note removed: "OreSat Proto-Card"
- title: (none) -> oresat-proto-card
- moved on the sheet: D3, Q2, Q9, R3, R70, R73, TP24, TP31

Commit message: Finished cleaning up protocard
Parts:
- C1, C16, C9: footprint oresat-proto-card:.0805-B-NOSILK -> oresat-passives:0805-B-NOSILK
- C11, C17, C22, C23, C3, C8, R17, R24, R3, R39, R40, R45, R46, R52, R53, R54, R55, R56, R57, R58, R59, R6, R60, R61, R62, R63, R65, R66, R67, R68, R69, R7, R70, R71, R72, R73, R74, R75, R76, R77, R78, R79, R80, R81, R82, R83: footprint oresat-proto-card:.0603-C-NOSILK -> oresat-passives:0603-C-NOSILK
- C2, C4, C5: symbol oresat-acs-card-eagle-import:C-EU0603-C-NOSILK -> oresat-proto-card-eagle-import:C-EU0603-C-NOSILK
- R1, R2, R4, R5: symbol oresat-acs-card-eagle-import:R-US_0603-C-NOSILK -> oresat-proto-card-eagle-import:R-US_0603-C-NOSILK
