File: m0-proto-card/m0-proto-card-sch-connectors.kicad_sch (KiCad schematic)
At the start: 13 parts, among them J1 J-SAMTEC-TFM-110-X1-XXX-D-RA, J2 U.FL, J3 U.FL, J4 U.FL, J6 J-SAMTEC-TFM-120-X1-XXX-D-RA

Commit message: More cleanup, and renaming of files, and better page layout
Other:
- title: oresat-proto-card -> OreSat M0 Proto Card: Connectors
Changed lines of the file:
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@@
 (kicad_sch (version 20230121) (generator eeschema)
-  (paper "B")
+  (paper "USLedger")
   (title_block
-    (title "oresat-proto-card")
-    (date "2024-02-25")
+    (title "OreSat M0 Proto Card: Connectors")
+    (date "2024-03-21")
     (rev "5.0")
   )
