File: m0-proto-card/m0-proto-card-sch-microcontroller.kicad_sch (KiCad schematic)
At the start: 25 parts, among them J7 ORESAT-DEBUG-CONNECTOR-ALL, U1 TCAN330, U7 STM32F091C, X2 CRYSTAL-WITH-GND

Commit message: More cleanup, and renaming of files, and better page layout
Other:
- title: oresat-proto-card -> OreSat M0 Proto Card: Microcontroller
- moved on the sheet: C13, C14, C15, C18, C19, C20, C21, D5, JP11, JP8, R47, R48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
