File: m0-proto-card/m0-proto-card-sch-power.kicad_sch (KiCad schematic)
At the start: 90 parts, among them Q1 MOSFET-PCH-SOT23-6, Q2 MOSFET-PCH-SOT23-6, Q7 MOSFET-PCH-SOT23-6, Q8 PMV45EN, Q9 PMV45EN, U10 TPS62111RSA, U11 MIC842LYC5, U12 MIC842LYC5, U2 MAX7310, U3 TS5A21366DCUR, U6 MAX4211

Commit message: More cleanup, and renaming of files, and better page layout
Other:
- title: oresat-proto-card -> OreSat M0 Proto Card: Power
- moved on the sheet: C1, C11, C16, C17, C2, C22, C23, C3, C4, C5, C8, C9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
