File: mcxn-proto-card/oresat-proto-card.kicad_pcb (KiCad board)
At the start: 4 copper layers, 99.8 x 94.6 mm, 201 parts, among them J1 J-SAMTEC-TFM-120-X1-XXX-D-RA, J2 J-SAMTEC-TFM-110-01-L-D-RA, J3 SM14B-SHLS-TF, J4 2477330-1, J5 2477330-1, J6 2477330-1, J7 U.FL-R-SMT-1(10), J8 U.FL-R-SMT-1(10), J9 U.FL-R-SMT-1(10), Q1 DMP2240UDM, Q2 DMP3050LVT-7, Q7 DMP3050LVT-7, Q8 PMV45EN, Q9 PMV45EN, U1 MCXN947VKLT, U10 TPS62111RSA, U11 MIC842LYC5, U12 MIC842LYC5, U2 MAX7310, U3 TS5A21366DCUR, U6 MAX4211FETE, U8 TCAN330, Y2 24 MHz

Commit message: Small cleanups for manufacturing
Parts:
- added FID1: Fiducial, Fiducial:Fiducial_1mm_Mask2mm, F.Cu at (103.0, 144.0)
- added FID2: Fiducial, Fiducial:Fiducial_1mm_Mask2mm, F.Cu at (192.0, 61.0)
- added FID3: Fiducial, Fiducial:Fiducial_1mm_Mask2mm, F.Cu at (192.0, 144.0)
- Q1: value DMP2240UDM -> DMP2110UVTQ-7
- Q2, Q7: value DMP3050LVT-7 -> DMPH2040UVTQ-7
- Q8, Q9: value PMV45EN -> DMN2050LQ-7
- moved TP6 1.47 mm to (125.3, 141.5)
- moved D4 0.98 mm to (139.4, 144.7)
- moved R21 0.98 mm to (139.4, 142.0)
- moved D3 0.98 mm to (136.1, 144.7)
- moved D6 0.98 mm to (137.8, 144.7)
- moved D7 0.98 mm to (134.5, 144.7)
- moved R17 0.98 mm to (137.8, 142.0)
- moved R3 0.98 mm to (136.1, 142.0)
- moved R76 0.98 mm to (134.5, 142.0)
Routing:
- net Net-(J3-DEBUG-0): track 1.71 -> 3.06 mm
- net +3.3V: track 44.9 -> 46.0 mm
- net /OreSat Power Domain/ON/~{OFF}: track 118.5 -> 119.3 mm
- net VBUSP: track 3.47 -> 2.67 mm
- net GND: vias 351 -> 350
- net (no net): vias 613 -> 614
